Commit message: 完成miniBox机器人大致的架构

File: robot/miniBox.urdf (robot description, URDF)
Before this commit: robot miniBox, 3 links, 2 joints
Links:
- added link front_follow_wheel, mass 0.3; collision cylinder length=0.05 radius=0.035; visual cylinder length=0.05 radius=0.035
- added link front_follow_wheel_pillar, mass 0.2; collision cylinder length=0.03 radius=0.075; visual cylinder length=0.03 radius=0.075
- link base_link: geometry collision box size=0.2 0.03 0.03; collision box size=0.2 0.03 0.03
Joints:
- added joint base_to_front_follow_wheel_pillar: type continuous, parent base_link, child front_follow_wheel_pillar, origin xyz=0.35 0 -0.115 rpy=0 0 0, axis 0 0 1
- added joint front_pillar_to_front_follow_wheel: type continuous, parent front_follow_wheel_pillar, child front_follow_wheel, origin xyz=0 0 -0.05 rpy=1.57075 0 0, axis 0 0 1
- joint joint_left_wheel: origin xyz=0 0.30 0 rpy=0 0 0 -> xyz=-0.1 0.30 0 rpy=0 0 0
- joint joint_right_wheel: origin xyz=0 -0.30 0 rpy=0 0 0 -> xyz=-0.1 -0.30 0 rpy=0 0 0
